Commit message: fix: align TOE foot geometry
变更内容：
- Correct the RR foot inertial, visual, collision, and fixed-joint origins in the URDF and MuJoCo assets.
- Assign stable names to all four MuJoCo foot collision geoms for runtime diagnostics.

File: resources/robots/TOE_dog4.5/urdf/dog.urdf (robot description, URDF)
Before this commit: robot TOE_dog4.5, 25 links, 24 joints
Joints:
- joint RR_foot_joint: origin xyz=0.016139 0 -0.18278 rpy=0 0 0 -> xyz=0.00070371 0 -0.21118 rpy=0 0 0

Commit message: chore: update Go2 policy and foot collision assets
变更内容：
- Update the deployed MNN policy and select the Sep16 training checkpoint for playback.
- Shift and narrow all four lower-leg collision cylinders to match the revised foot geometry.

File: resources/robots/TOE_dog4.5/urdf/dog.urdf (robot description, URDF)
Before this commit: robot TOE_dog4.5, 25 links, 24 joints
Links:
- link FL_calflower1: geometry collision cylinder length=0.03 radius=0.014
- link FR_calflower1: geometry collision cylinder length=0.03 radius=0.014
- link RL_calflower1: geometry collision cylinder length=0.03 radius=0.014
- link RR_calflower1: geometry collision cylinder length=0.03 radius=0.014
